File: Accelerometer/Accelerometer.kicad_sch (KiCad schematic)
At the start: 14 parts, among them U1 DA14531_17-ball_WLCSP, U2 LIS2DU12, Y1 Crystal_GND24

Commit message: Double checked schematic
Parts:
- added C3: C, Capacitor_SMD:C_0201_0603Metric, symbol Device:C
- added TP4: +Ve charging, symbol Connector:TestPoint
- added TP5: Gnd charging, symbol Connector:TestPoint
Connections:
- net at C1.2, C2.2, D1.1 (K)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: now also U2.3 (SDO/SA0), C3.2, TP5.1
- net at +ve1.1, C1.1, C2.1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: now also C3.1, TP4.1; no longer U2.3 (SDO/SA0)
Other:
- moved on the sheet: C1, C2, U2
